File: adf7021_module.sch (KiCad schematic (older format))
At the start: 71 parts, among them J1 Conn_02x10_Counter_Clockwise, J2 Conn_Coaxial, J3 Conn_Coaxial, J4 Conn_02x10_Counter_Clockwise, U1 ADF7021, X1 19.68MHz

Commit message: Adding bus resistors on all inputs / outputs
You get a bus resistor! You get a bus resistor!

EVERYONE GETS A BUS RESISTOOOOORRR!!1
Parts:
- added R19, R20, R21, R22, R23, R24: 22, symbol Device:R
- gave numbers to parts that had none: 4
Connections:
- net CE: now also R17.2, R21.2; no longer J1.3 (Pin_3), J4.3 (Pin_3)
- net CLKOUT: now also R16.1; no longer R14.1
- net MUXOUT: now also R15.1; no longer U1.37 (MUXOUT)
- net SCLK: now also R20.2, R24.2; no longer R16.2, R18.2
- net SDATA: now also R19.2, R23.2; no longer R15.2, R17.2
- net SLE: now also R18.2, R22.2; no longer J1.4 (Pin_4), J4.4 (Pin_4)
- net SWD: now also R14.1; no longer U1.33 (SWD)
- net at R14.2: now also U1.33 (SWD); no longer U1.36 (CLKOUT)
- net at J1.6 (Pin_6): now also R19.1; no longer R15.1
- net at J1.7 (Pin_7): now also R20.1; no longer R16.1
- net at R17.1: now also J1.3 (Pin_3); no longer J4.6 (Pin_6)
- net at R18.1: now also J1.4 (Pin_4); no longer J4.7 (Pin_7)
- new net: R16.2, U1.36 (CLKOUT)
- new net: R15.2, U1.37 (MUXOUT)
- new net: J4.3 (Pin_3), R21.1
- new net: J4.4 (Pin_4), R22.1
- new net: J4.6 (Pin_6), R23.1
- new net: J4.7 (Pin_7), R24.1
Other:
- moved on the sheet: R14, R15, R16, R17, R18
Changed lines of the file:
@@
 	5400 3200 5050 3200
 Wire Wire Line
-	4600 3100 5400 3100
-Wire Wire Line
-	5400 3000 4600 3000
+	4600 3100 4750 3100
+Wire Wire Line
+	5400 3000 5050 3000
 Wire Wire Line
 	4600 2900 4750 2900
@@
 Text GLabel 11000 7050 0    50   Input ~ 0
 SDATA
-Text GLabel 11250 6850 0    50   Input ~ 0
+Text GLabel 11000 6850 0    50   Input ~ 0
 SLE
-Text GLabel 11250 6750 0    50   Input ~ 0
+Text GLabel 11000 6750 0    50   Input ~ 0
 CE
 Text GLabel 12350 7150 2    50   BiDi ~ 0
@@
 Text GLabel 12350 7450 2    50   Output ~ 0
 CLKOUT
-Text GLabel 11250 6650 0    50   Input ~ 0
+Text GLabel 11000 6650 0    50   Input ~ 0
 FM_MOD
 Text GLabel 11400 7450 0    50   Input ~ 0
@@
 $EndComp
 Wire Wire Line
-	11250 6750 11550 6750
-Wire Wire Line
-	11550 6850 11250 6850
+	11000 6750 11100 6750
+Wire Wire Line
+	11550 6850 11400 6850
 Wire Wire Line
 	12050 6850 12350 6850
@@
 	2700 2950 1950 2950
 Wire Wire Line
-	11550 6650 11250 6650
+	11550 6650 11000 6650
 $Comp
 L power:+3V3 #PWR?
@@
 Text GLabel 11000 8400 0    50   Input ~ 0
 SDATA
-Text GLabel 11250 8200 0    50   Input ~ 0
+Text GLabel 11000 8200 0    50   Input ~ 0
 SLE
-Text GLabel 11250 8100 0    50   Input ~ 0
+Text GLabel 11000 8100 0    50   Input ~ 0
 CE
 Text GLabel 12350 8500 2    50   BiDi ~ 0
@@
 $EndComp
 Wire Wire Line
-	11250 8100 11550 8100
-Wire Wire Line
-	11550 8200 11250 8200
+	11000 8100 11100 8100
+Wire Wire Line
+	11550 8200 11400 8200
 Wire Wire Line
 	12050 8200 12350 8200
@@
 Wire Wire Line
 	11450 8600 11550 8600
-Text Notes 10650 6850 1    30   ~ 0
+Text Notes 10600 6850 1    30   ~ 0
 Analog\nLow Speed
-Text Notes 10650 7200 1    30   ~ 0
+Text Notes 10600 7200 1    30   ~ 0
 Data / SPI
-Text Notes 10650 7500 1    30   ~ 0
+Text Notes 10600 7500 1    30   ~ 0
 Clocks
 $Comp
 L Device:R R14
 U 1 1 60677D63
-P 4900 3200
-F 0 "R14" V 4850 3400 50  0000 C CNN
-F 1 "22" V 4900 3200 50  0000 C CNN
-F 2 "" V 4830 3200 50  0001 C CNN
-F 3 "~" H 4900 3200 50  0001 C CNN
-	1    4900 3200
+P 4900 3000
+F 0 "R14" V 4850 3200 50  0000 C CNN
+F 1 "22" V 4900 3000 50  0000 C CNN
+F 2 "" V 4830 3000 50  0001 C CNN
+F 3 "~" H 4900 3000 50  0001 C CNN
+	1    4900 3000
 	0    1    1    0
 $EndComp
@@
 L Device:R R17
 U 1 1 6070C2A8
+P 11250 6750
+F 0 "R17" V 11200 6950 50  0000 C CNN
+F 1 "22" V 11250 6750 50  0000 C CNN
+F 2 "" V 11180 6750 50  0001 C CNN
+F 3 "~" H 11250 6750 50  0001 C CNN
+	1    11250 6750
+	0    1    1    0
+$EndComp
+Wire Wire Line
+	11400 8400 11550 8400
+$Comp
+L Device:R R18
+U 1 1 60741E3A
+P 11250 6850
+F 0 "R18" V 11200 7050 50  0000 C CNN
+F 1 "22" V 11250 6850 50  0000 C CNN
+F 2 "" V 11180 6850 50  0001 C CNN
+F 3 "~" H 11250 6850 50  0001 C CNN
+	1    11250 6850
+	0    1    1    0
+$EndComp
+Wire Wire Line
+	11400 8500 11550 8500
+$Comp
+L Device:R R15
+U 1 1 607BA8AF
+P 4900 3100
+F 0 "R15" V 4850 3300 50  0000 C CNN
+F 1 "22" V 4900 3100 50  0000 C CNN
+F 2 "" V 4830 3100 50  0001 C CNN
+F 3 "~" H 4900 3100 50  0001 C CNN
+	1    4900 3100
+	0    1    1    0
+$EndComp
+Wire Wire Line
+	11400 7050 11550 7050
+$Comp
+L Device:R R16
+U 1 1 607BB020
+P 4900 3200
+F 0 "R16" V 4850 3400 50  0000 C CNN
+F 1 "22" V 4900 3200 50  0000 C CNN
+F 2 "" V 4830 3200 50  0001 C CNN
+F 3 "~" H 4900 3200 50  0001 C CNN
+	1    4900 3200
+	0    1    1    0
+$EndComp
+Wire Wire Line
+	11400 7150 11550 7150
+Connection ~ 11600 4400
+Wire Wire Line
+	12150 4400 12350 4400
+Wire Wire Line
+	11600 3700 11600 3300
+Wire Wire Line
+	11050 3300 11600 3300
+$Comp
+L Mechanical:MountingHole_Pad H1
+U 1 1 608F38E7
+P 14150 8200
+F 0 "H1" H 14250 8203 50  0000 L CNN
+F 1 "MountingHole_Pad" H 14250 8158 50  0001 L CNN
+F 2 "" H 14150 8200 50  0001 C CNN
+F 3 "~" H 14150 8200 50  0001 C CNN
+	1    14150 8200
+	1    0    0    -1
+$EndComp
+$Comp
+L Mechanical:MountingHole_Pad H2
+U 1 1 608F437B
+P 14550 8200
+F 0 "H2" H 14650 8203 50  0000 L CNN
+F 1 "MountingHole_Pad" H 14650 8158 50  0001 L CNN
+F 2 "" H 14550 8200 50  0001 C CNN
+F 3 "~" H 14550 8200 50  0001 C CNN
+	1    14550 8200
+	1    0    0    -1
+$EndComp
+$Comp
+L Mechanical:MountingHole_Pad H3
+U 1 1 608F497B
+P 14950 8200
+F 0 "H3" H 15050 8203 50  0000 L CNN
+F 1 "MountingHole_Pad" H 15050 8158 50  0001 L CNN
+F 2 "" H 14950 8200 50  0001 C CNN
+F 3 "~" H 14950 8200 50  0001 C CNN
+	1    14950 8200
+	1    0    0    -1
+$EndComp
+$Comp
+L Mechanical:MountingHole_Pad H4
+U 1 1 608F4F4D
+P 15350 8200
+F 0 "H4" H 15450 8203 50  0000 L CNN
+F 1 "MountingHole_Pad" H 15450 8158 50  0001 L CNN
+F 2 "" H 15350 8200 50  0001 C CNN
+F 3 "~" H 15350 8200 50  0001 C CNN
+	1    15350 8200
+	1    0    0    -1
+$EndComp
+$Comp
+L power:GND #PWR040
+U 1 1 608F5BFE
+P 14150 8500
+F 0 "#PWR040" H 14150 8250 50  0001 C CNN
+F 1 "GND" H 14155 8327 50  0000 C CNN
+F 2 "" H 14150 8500 50  0001 C CNN
+F 3 "" H 14150 8500 50  0001 C CNN
+	1    14150 8500
+	1    0    0    -1
+$EndComp
+Wire Wire Line
+	14150 8500 14150 8400
+Wire Wire Line
+	14150 8400 14550 8400
+Wire Wire Line
+	15350 8400 15350 8300
+Connection ~ 14150 8400
+Wire Wire Line
+	14150 8400 14150 8300
+Wire Wire Line
+	14950 8300 14950 8400
+Connection ~ 14950 8400
+Wire Wire Line
+	14950 8400 15350 8400
+Wire Wire Line
+	14550 8300 14550 8400
+Connection ~ 14550 8400
+Wire Wire Line
+	14550 8400 14950 8400
+Wire Wire Line
+	4750 3000 4600 3000
+Wire Wire Line
+	5050 3100 5400 3100
+$Comp
+L Device:R R22
+U 1 1 6095F1AE
+P 11250 8200
+F 0 "R22" V 11200 8400 50  0000 C CNN
+F 1 "22" V 11250 8200 50  0000 C CNN
+F 2 "" V 11180 8200 50  0001 C CNN
+F 3 "~" H 11250 8200 50  0001 C CNN
+	1    11250 8200
+	0    1    1    0
+$EndComp
+$Comp
+L Device:R R21
+U 1 1 6095EF74
+P 11250 8100
+F 0 "R21" V 11200 8300 50  0000 C CNN
+F 1 "22" V 11250 8100 50  0000 C CNN
+F 2 "" V 11180 8100 50  0001 C CNN
+F 3 "~" H 11250 8100 50  0001 C CNN
+	1    11250 8100
+	0    1    1    0
+$EndComp
+$Comp
+L Device:R R20
+U 1 1 609DA120
+P 11250 7150
+F 0 "R20" V 11200 7350 50  0000 C CNN
+F 1 "22" V 11250 7150 50  0000 C CNN
+F 2 "" V 11180 7150 50  0001 C CNN
+F 3 "~" H 11250 7150 50  0001 C CNN
+	1    11250 7150
+	0    1    1    0
+$EndComp
+Wire Wire Line
+	11100 6850 11000 6850
+$Comp
+L Device:R R19
+U 1 1 609DA9F4
+P 11250 7050
+F 0 "R19" V 11200 7250 50  0000 C CNN
+F 1 "22" V 11250 7050 50  0000 C CNN
+F 2 "" V 11180 7050 50  0001 C CNN
+F 3 "~" H 11250 7050 50  0001 C CNN
+	1    11250 7050
+	0    1    1    0
+$EndComp
+Wire Wire Line
+	11400 6750 11550 6750
+$Comp
+L Device:R R24
+U 1 1 60A0D87B
+P 11250 8500
+F 0 "R24" V 11200 8700 50  0000 C CNN
+F 1 "22" V 11250 8500 50  0000 C CNN
+F 2 "" V 11180 8500 50  0001 C CNN
+F 3 "~" H 11250 8500 50  0001 C CNN
+	1    11250 8500
+	0    1    1    0
+$EndComp
+Wire Wire Line
+	11100 8200 11000 8200
+$Comp
+L Device:R R23
+U 1 1 60A0DCBE
 P 11250 8400
-F 0 "R17" V 11200 8600 50  0000 C CNN
+F 0 "R23" V 11200 8600 50  0000 C CNN
 F 1 "22" V 11250 8400 50  0000 C CNN
 F 2 "" V 11180 8400 50  0001 C CNN
@@
 $EndComp
 Wire Wire Line
-	11400 8400 11550 8400
-$Comp
-L Device:R R18
-U 1 1 60741E3A
-P 11250 8500
-F 0 "R18" V 11200 8700 50  0000 C CNN
-F 1 "22" V 11250 8500 50  0000 C CNN
-F 2 "" V 11180 8500 50  0001 C CNN
-F 3 "~" H 11250 8500 50  0001 C CNN
-	1    11250 8500
-	0    1    1    0
-$EndComp
-Wire Wire Line
-	11400 8500 11550 8500
-$Comp
-L Device:R R15
-U 1 1 607BA8AF
-P 11250 7050
-F 0 "R15" V 11200 7250 50  0000 C CNN
-F 1 "22" V 11250 7050 50  0000 C CNN
-F 2 "" V 11180 7050 50  0001 C CNN
-F 3 "~" H 11250 7050 50  0001 C CNN
-	1    11250 7050
-	0    1    1    0
-$EndComp
-Wire Wire Line
-	11400 7050 11550 7050
-$Comp
-L Device:R R16
-U 1 1 607BB020
-P 11250 7150
-F 0 "R16" V 11200 7350 50  0000 C CNN
-F 1 "22" V 11250 7150 50  0000 C CNN
-F 2 "" V 11180 7150 50  0001 C CNN
-F 3 "~" H 11250 7150 50  0001 C CNN
-	1    11250 7150
-	0    1    1    0
-$EndComp
-Wire Wire Line
-	11400 7150 11550 7150
-Connection ~ 11600 4400
-Wire Wire Line
-	12150 4400 12350 4400
-Wire Wire Line
-	11600 3700 11600 3300
-Wire Wire Line
-	11050 3300 11600 3300
-$Comp
-L Mechanical:MountingHole_Pad H?
-U 1 1 608F38E7
-P 14150 8200
-F 0 "H?" H 14250 8203 50  0000 L CNN
-F 1 "MountingHole_Pad" H 14250 8158 50  0001 L CNN
-F 2 "" H 14150 8200 50  0001 C CNN
-F 3 "~" H 14150 8200 50  0001 C CNN
-	1    14150 8200
-	1    0    0    -1
-$EndComp
-$Comp
-L Mechanical:MountingHole_Pad H?
-U 1 1 608F437B
-P 14550 8200
-F 0 "H?" H 14650 8203 50  0000 L CNN
-F 1 "MountingHole_Pad" H 14650 8158 50  0001 L CNN
-F 2 "" H 14550 8200 50  0001 C CNN
-F 3 "~" H 14550 8200 50  0001 C CNN
-	1    14550 8200
-	1    0    0    -1
-$EndComp
-$Comp
-L Mechanical:MountingHole_Pad H?
-U 1 1 608F497B
-P 14950 8200
-F 0 "H?" H 15050 8203 50  0000 L CNN
-F 1 "MountingHole_Pad" H 15050 8158 50  0001 L CNN
-F 2 "" H 14950 8200 50  0001 C CNN
-F 3 "~" H 14950 8200 50  0001 C CNN
-	1    14950 8200
-	1    0    0    -1
-$EndComp
-$Comp
-L Mechanical:MountingHole_Pad H?
-U 1 1 608F4F4D
-P 15350 8200
-F 0 "H?" H 15450 8203 50  0000 L CNN
-F 1 "MountingHole_Pad" H 15450 8158 50  0001 L CNN
-F 2 "" H 15350 8200 50  0001 C CNN
-F 3 "~" H 15350 8200 50  0001 C CNN
-	1    15350 8200
-	1    0    0    -1
-$EndComp
-$Comp
-L power:GND #PWR?
-U 1 1 608F5BFE
-P 14150 8500
-F 0 "#PWR?" H 14150 8250 50  0001 C CNN
-F 1 "GND" H 14155 8327 50  0000 C CNN
-F 2 "" H 14150 8500 50  0001 C CNN
-F 3 "" H 14150 8500 50  0001 C CNN
-	1    14150 8500
-	1    0    0    -1
-$EndComp
-Wire Wire Line
-	14150 8500 14150 8400
-Wire Wire Line
-	14150 8400 14550 8400
-Wire Wire Line
-	15350 8400 15350 8300
-Connection ~ 14150 8400
-Wire Wire Line
-	14150 8400 14150 8300
-Wire Wire Line
-	14950 8300 14950 8400
-Connection ~ 14950 8400
-Wire Wire Line
-	14950 8400 15350 8400
-Wire Wire Line
-	14550 8300 14550 8400
-Connection ~ 14550 8400
-Wire Wire Line
-	14550 8400 14950 8400
+	11400 8100 11550 8100
 $EndSCHEMATC

Commit message: rough component placement, stackup definition
Parts:
- C1, C10, C11, C12, C13, C14, C15, C16, C17, C18, C19, C2, C20, C21, C22, C23, C24, C25, C26, C27, C28, C29, C3, C30, C31, C32, C33, C4, C5, C6, C7, C8, C9: footprint (none) -> Capacitor_SMD:C_0402_1005Metric_Pad0.74x0.62mm_HandSolder
- C34, C35, C36: footprint (none) -> Capacitor_SMD:C_0603_1608Metric_Pad1.08x0.95mm_HandSolder
- H1, H2, H3, H4: footprint (none) -> MountingHole:MountingHole_3.2mm_M3_DIN965_Pad_TopBottom
- J1: footprint (none) -> Connector_Hirose:Hirose_DF12_DF12E3.0-20DP-0.5V_2x10_P0.50mm_Vertical
- J2, J3: footprint (none) -> Connector_Coaxial:SMA_Molex_73251-2200_Horizontal
- J4: footprint (none) -> Connector_PinSocket_2.54mm:PinSocket_2x10_P2.54mm_Vertical
- L1, L2, L3, L4, L5, L6, L7: footprint (none) -> Inductor_SMD:L_0402_1005Metric_Pad0.77x0.64mm_HandSolder
- R1, R10, R11, R12, R13, R14, R15, R16, R17, R18, R19, R2, R20, R21, R22, R23, R24, R3, R4, R5, R6, R7, R8, R9: footprint (none) -> Resistor_SMD:R_0402_1005Metric_Pad0.72x0.64mm_HandSolder

Commit message: some more layout attempts
Parts:
- removed R11, R12, R15, R16, R17, R18, R19, R20, R21, R22, R23, R24: 22, Resistor_SMD:R_0402_1005Metric_Pad0.72x0.64mm_HandSolder, symbol Device:R
- added RN1, RN2, RN3: 22, Resistor_SMD:R_Array_Concave_4x0402, symbol Device:R_Pack04_Split
- H1, H2, H3, H4: footprint MountingHole:MountingHole_3.2mm_M3_DIN965_Pad_TopBottom -> MountingHole:MountingHole_2.2mm_M2_Pad_TopBottom
- J1: symbol Connector_Generic:Conn_02x10_Counter_Clockwise -> Connector_Generic:Conn_02x10_Top_Bottom
- J4: symbol Connector_Generic:Conn_02x10_Counter_Clockwise -> Connector_Generic:Conn_02x10_Odd_Even
- R13: value 22 -> 1k
Connections:
- net +3V3: now also J1.10 (Pin_10), J4.19 (Pin_19); no longer J1.1 (Pin_1), J4.1 (Pin_1)
- net ADCIN: now also J4.18 (Pin_18); no longer J4.19 (Pin_19)
- net CE: now also RN2.4 (R4.1), RN3.4 (R4.1)
- net CLKOUT: now also J4.2 (Pin_2), R13.1; no longer J4.11 (Pin_11)
- net CLK_IN: now also J1.1 (Pin_1), J4.1 (Pin_1); no longer J1.10 (Pin_10), J4.10 (Pin_10)
- net FM_MOD: now also J1.9 (Pin_9), J4.17 (Pin_17); no longer J1.2 (Pin_2), J4.2 (Pin_2)
- net GND: now also J1.2 (Pin_2), J1.3 (Pin_3), J1.6 (Pin_6), J4.11 (Pin_11), J4.3 (Pin_3), J4.4 (Pin_4); no longer J1.5 (Pin_5), J1.8 (Pin_8), J1.9 (Pin_9), J4.16 (Pin_16), J4.8 (Pin_8), J4.9 (Pin_9)
- net MUXOUT: now also J4.14 (Pin_14), RN1.8 (R1.2); no longer J4.17 (Pin_17)
- net SCLK: now also RN2.1 (R1.1), RN3.1 (R1.1)
- net SDATA: now also RN2.2 (R2.1), RN3.2 (R2.1)
- net SLE: now also RN2.3 (R3.1), RN3.3 (R3.1)
- net SREAD: now also J4.10 (Pin_10), R14.1; no longer J4.15 (Pin_15), R13.1
- net SWD: now also J4.16 (Pin_16), RN1.5 (R4.2); no longer J4.18 (Pin_18), R14.1
- net TxRxCLK: now also J4.6 (Pin_6), RN1.7 (R2.2); no longer J4.13 (Pin_13)
- net TxRxData: now also J4.8 (Pin_8), RN1.6 (R3.2); no longer J4.14 (Pin_14)
- net at U1.27 (SREAD): now also R14.2; no longer R13.2
- net at U1.33 (SWD): now also RN1.4 (R4.1); no longer R14.2
- net at U1.34 (TxRxDATA): now also RN1.3 (R3.1)
- net at U1.35 (TxRxCLK): now also RN1.2 (R2.1)
- net at U1.36 (CLKOUT): now also R13.2
- net at U1.37 (MUXOUT): now also RN1.1 (R1.1)
- net at J1.4 (Pin_4): now also RN2.8 (R1.2)
- net at J1.7 (Pin_7): now also RN2.6 (R3.2)
- net at J4.7 (Pin_7): now also RN3.8 (R1.2)
- new net: J1.8 (Pin_8), RN2.5 (R4.2)
- new net: J1.5 (Pin_5), RN2.7 (R2.2)
- new net: J4.13 (Pin_13), RN3.6 (R3.2)
- new net: J4.15 (Pin_15), RN3.5 (R4.2)
- new net: J4.9 (Pin_9), RN3.7 (R2.2)
Other:
- moved on the sheet: C34, C35, C36, H1, H2, H3, H4, J1, J4, R13, R14
